Commit message: A big hack to change all joints to fixed

File: robots/robotiq_arg85_description.URDF (robot description, URDF)
Before this commit: robot robotiq_arg85_description, 9 links, 8 joints
Joints:
- joint finger_joint: type revolute -> fixed
- joint left_inner_finger_joint: type revolute -> fixed
- joint left_inner_knuckle_joint: type revolute -> fixed
- joint right_inner_finger_joint: type revolute -> fixed
- joint right_inner_knuckle_joint: type revolute -> fixed
- joint right_outer_knuckle_joint: type revolute -> fixed
